File: kicad/Power.kicad_sch (KiCad schematic)
At the start: 18 parts, among them J7 10137064-00021LF, J8 Conn_01x06_Pin, Q4 Si2319CDS, Q5 Si2319CDS, U2 CYPD3177-24LQ

Commit message: finalized pcb
Parts:
- removed J7: 10137064-00021LF, 10137064-00021LF:AMPHENOL_10137064-00021LF, symbol 10137064-00021LF:10137064-00021LF
- added J10: 10137064-00021LF, Ampheon-10137064-00021LF:AMPHENOL_10137064-00021LF, symbol 10137064-00021LF:10137064-00021LF
- R9: footprint (none) -> Resistor_SMD:R_0603_1608Metric
Connections:
- net CC1: now also J10.A5 (CC1)
- net CC2: now also J10.B5 (CC2)
- net GND: now also J10.A1 (GND_A), J10.A12 (GND_A__1), J10.B1 (GND_B), J10.B12 (GND_B__1), J10.SH1 (SHIELD), J10.SH2 (SHIELD__1), J10.SH3 (SHIELD__2), J10.SH4 (SHIELD__4)
- net VBUS: now also J10.A4 (VBUS_A), J10.B4 (VBUS_B)
- net at R10.1, U2.13 (HPI_SCL): now also J8.6 (Pin_6); no longer J8.5 (Pin_5)
- net at R13.1, U2.8 (GPIO_1): now also J8.2 (Pin_2); no longer J8.1 (Pin_1)
- net at U2.9 (FAULT): now also J8.3 (Pin_3); no longer J8.2 (Pin_2)
- net at R12.1, U2.7 (~{HPI_INT}): now also J8.1 (Pin_1); no longer J8.3 (Pin_3)
- net at R11.1, U2.12 (HPI_SDA): now also J8.5 (Pin_5); no longer J8.4 (Pin_4)
- net at R9.1, U2.10 (FLIP): now also J8.4 (Pin_4); no longer J8.6 (Pin_6)

Commit message: feat: v2
Parts:
- removed J10: 10137064-00021LF, Ampheon-10137064-00021LF:AMPHENOL_10137064-00021LF, symbol 10137064-00021LF:10137064-00021LF
- removed J8: Conn_01x06_Pin, Connector_PinHeader_2.54mm:PinHeader_1x06_P2.54mm_Vertical, symbol Connector:Conn_01x06_Pin
- removed Q4: Si2319CDS, Package_TO_SOT_SMD:SOT-23-3, symbol Transistor_FET:Si2343CDS
- removed Q5: Si2319CDS, Package_TO_SOT_SMD:SOT-23, symbol Transistor_FET:Si2329CDS
- added C12: 10uF, Capacitor_SMD:C_0603_1608Metric, symbol Device:C
- added C13, C17: 4.7uF, Capacitor_SMD:C_0603_1608Metric, symbol Device:C
- added C14, C15, C16: 22uF, Capacitor_SMD:C_0805_2012Metric, symbol Device:C
- added C18, C26: 2.2uF, Capacitor_SMD:C_0603_1608Metric, symbol Device:C
- added C22, C23: 1uF, Capacitor_SMD:C_0805_2012Metric, symbol Device:C
- added C24: 10uF, Capacitor_SMD:C_0805_2012Metric, symbol Device:C
- added C25: 0.1uF, Resistor_SMD:R_0402_1005Metric, symbol Device:C
- added D1: B340B-13-F, Diode_SMD:D_SMB, symbol Device:D_Schottky
- added J10: UJ40-C-H-G-SMT-P24-TR, Own:SAMESKY_UJ40-C-H-G-SMT-P24-TR, symbol UJ40-C-H-G-SMT-P24-TR:UJ40-C-H-G-SMT-P24-TR
- added L1: 4.7uH, Own:IND_NRS5030T100MMGJ_TAY, symbol Device:L
- added L2: 3.3-4.7uH, Inductor_SMD:L_Coilcraft_XxL4030, symbol Device:L
- added Q3, Q4: FDS8949, Own:SOIC8_3P9X4P9_OSI, symbol FDS8949:FDS8949
- added R15: 10k, Capacitor_SMD:C_0603_1608Metric, symbol Device:R
- added R16: 50k, Resistor_SMD:R_0603_1608Metric, symbol Device:R
- added R17: 1k, Capacitor_SMD:C_0603_1608Metric, symbol Device:R
- added R18: 1k, Resistor_SMD:R_0402_1005Metric, symbol Device:R
- added R19: 49.9k, Resistor_SMD:R_0402_1005Metric, symbol Device:R
- added U1: TS30013-M033QFNR, Own:QFN16_3X3_SEM, symbol TS30011-M033QFNR:TS30013-M033QFNR
- added U3: MAX26405AFOAY+T, Own:FC2QFN-17, symbol Own:MAX26405AFOAY+T
- C10, C11, C8: footprint Capacitor_SMD:C_0603_1608Metric -> Capacitor_SMD:C_0402_1005Metric
- C9: footprint Resistor_SMD:R_0603_1608Metric -> Capacitor_SMD:C_0402_1005Metric
- R10, R11, R12, R9: footprint Resistor_SMD:R_0603_1608Metric -> Resistor_SMD:R_0402_1005Metric
- R13: value 2.2k -> 10k; footprint Resistor_SMD:R_0603_1608Metric -> Resistor_SMD:R_0402_1005Metric
- R5: value R -> bridge; footprint Resistor_SMD:R_0603_1608Metric -> Resistor_SMD:R_0402_1005Metric
- R6, R8: value R -> 5.1k; footprint Resistor_SMD:R_0603_1608Metric -> Resistor_SMD:R_0402_1005Metric
- R7: value R -> dont connect; footprint Resistor_SMD:R_0603_1608Metric -> Resistor_SMD:R_0402_1005Metric
Connections:
- net +3.3V: no longer R10.2, R11.2, R12.2, R13.2
- net +5V: now also C14.2, C15.2, C16.2, L2.1, Q4.3, U3.13 (OUT)
- net CC1: now also J10.A5 (CC1)
- net CC2: now also J10.B5 (CC2)
- net GND: now also R10.2, R11.2, R12.2, C13.2, C14.1, C15.1, C16.1, C17.1, C18.2, C24.1, J10.A1 (GND), J10.A12 (GND__1), J10.B1 (GND__2), J10.B12 (GND__3), J10.SH1 (SHIELD), J10.SH10 (SHIELD__9), J10.SH2 (SHIELD__1), J10.SH3 (SHIELD__2), J10.SH4 (SHIELD__3), J10.SH5 (SHIELD__4), J10.SH6 (SHIELD__5), J10.SH7 (SHIELD__6), J10.SH8 (SHIELD__7), J10.SH9 (SHIELD__8), U1.14 (PGND), U1.15 (PGND), U1.17 (EPAD), U1.4 (GND), U3.10 (GND), U3.5 (PGND), U3.7 (PGND)
- net VBUS: now also C22.1, C24.2, D1.2 (A), J10.A4 (VBUS), J10.A9 (VBUS__1), J10.B4 (VBUS__2), J10.B9 (VBUS__3), Q3.1, Q4.1, R15.1, R16.2, R19.2
- net VD: now also C23.2, Q3.3, U1.11 (VCC), U1.2 (VCC), U1.3 (VCC), U1.9 (EN), U3.1 (EN)
- net I2C1_SCL: now reaches R10.1, U2.13 (HPI_SCL)
- net ~{HP INT}: now reaches R12.1, U2.7 (~{HPI_INT})
- net at R13.1: now also U1.8 (PG); no longer U2.8 (GPIO_1)
- net I2C1_SDA: now reaches R11.1, U2.12 (HPI_SDA)
- net SAFE PWR: now reaches U2.4 (SAFE_PWR_EN)
- net SAFE PWR: now also R18.2
- net at U2.3 (VBUS_FET_EN): now also R17.1
- new net: C25.1, L1.1, U1.1 (VSW), U1.12 (VSW), U1.13 (VSW), U1.16 (VSW)
- new net: C25.2, U1.10 (BST)
- new net: C22.2, C23.1, Q3.2, Q3.4, R15.2, R17.2
- new net: D1.1 (K), Q3.5, Q3.6, Q3.7, Q3.8, R16.1
- new net: C12.1, C26.1, U3.2 (BST)
- new net: C12.2, C26.2, L2.2, U3.6 (LX)
- new net: C17.2, U3.9 (SUP)
- new net: Q4.2, Q4.4, R18.1, R19.1
- new net: Q4.5, Q4.6, Q4.7, Q4.8
- new net: C18.1, U3.11 (BIAS), U3.12 (FB), U3.16 (SYNC)
- new net: C13.1, U3.3 (SUP)
- new net VDD: L1.2, R13.2, U1.5 (FB)
Other:
- moved on the sheet: R9

Commit message: fix: minor additions to v2
Other:
- company: (none) -> vividsystem
- title: (none) -> Painter HAT Power Supply
Changed lines of the file:
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@@
 	(generator_version "9.0")
 	(paper "A4")
+	(title_block
+		(title "Painter HAT Power Supply")
+		(rev "v2")
+		(company "vividsystem")
+	)
 	(junction
 		(at 48.26 39.37)

Commit message: feat: v2.1
Parts:
- removed J10: UJ40-C-H-G-SMT-P24-TR, Own:SAMESKY_UJ40-C-H-G-SMT-P24-TR, symbol UJ40-C-H-G-SMT-P24-TR:UJ40-C-H-G-SMT-P24-TR
- removed L2: 3.3-4.7uH, Inductor_SMD:L_Coilcraft_XxL4030, symbol Device:L
- removed U3: MAX26405AFOAY+T, Own:FC2QFN-17, symbol Own:MAX26405AFOAY+T
- added C29: 0.47uF, Capacitor_SMD:C_0402_1005Metric, symbol Device:C
- added C32: 1uF, Capacitor_SMD:C_0402_1005Metric, symbol Device:C
- added C33: 2.2uF, Capacitor_SMD:C_0402_1005Metric, symbol Device:C
- added L3: 5.2uH, easyeda2kicad:IND-SMD_4P-L10.5-W9.5-TL, symbol Device:L
- added R1: 100k, Resistor_SMD:R_0603_1608Metric, symbol Device:R
- added R2: 10k, Resistor_SMD:R_0402_1005Metric, symbol Device:R
- added R20: 24.9k, Resistor_SMD:R_0603_1608Metric, symbol Device:R
- added R3: 75k, Resistor_SMD:R_0603_1608Metric, symbol Device:R
- added R4: 4.07k, Resistor_SMD:R_0603_1608Metric, symbol Device:R
- added U5: LM76005RNPR, easyeda2kicad:WQFN-30_L6.0-W4.0-P0.50-TL-EP_LM76005RNPR, symbol easyeda2kicad:LM76005RNPR
- added USBC1: TYPE-C-31-M-12, easyeda2kicad:USB-C_SMD-TYPE-C-31-M-12, symbol easyeda2kicad:TYPE-C-31-M-12
- C12: footprint Capacitor_SMD:C_0603_1608Metric -> Capacitor_SMD:C_0805_2012Metric
- C13: value 4.7uF -> 10uF; footprint Capacitor_SMD:C_0603_1608Metric -> Capacitor_SMD:C_0805_2012Metric
- C14: value 22uF -> 100uF; footprint Capacitor_SMD:C_0805_2012Metric -> Capacitor_SMD:C_Elec_8x10.2
- C15, C16: value 22uF -> 47uF
- C17: value 4.7uF -> 47uF; footprint Capacitor_SMD:C_0603_1608Metric -> Capacitor_SMD:C_0805_2012Metric
- C18: value 2.2uF -> 10nF; footprint Capacitor_SMD:C_0603_1608Metric -> Capacitor_SMD:C_0402_1005Metric
- C25: value 0.1uF -> 100nF
- C26: value 2.2uF -> 100pF; footprint Capacitor_SMD:C_0603_1608Metric -> Capacitor_SMD:C_0402_1005Metric
- R7: value dont connect -> leave open
Connections:
- net +5V: now also C15.1, C16.1, C17.1, C26.1, C32.2, L3.1, R1.1, R2.1, U5.9 (BIAS); no longer C14.2, C15.2, C16.2
- net CC1: now also USBC1.A5 (CC1)
- net CC2: now also USBC1.B5 (CC2)
- net GND: now also C12.2, C14.2, C15.2, C16.2, C17.2, C32.1, C33.1, R20.2, R4.1, U5.13 (AGND), U5.14 (AGND), U5.15 (AGND), U5.17 (SYNC/MODE), U5.19 (NC), U5.24 (PGND), U5.25 (PGND), U5.26 (PGND), U5.27 (NC), U5.28 (NC), U5.29 (NC), U5.30 (NC), U5.31 (EP), USBC1.0 (SH), USBC1.A1 (GND), USBC1.A12 (GND), USBC1.B1 (GND), USBC1.B12 (GND); no longer C14.1, C15.1, C16.1, C17.1
- net VBUS: now also USBC1.A4 (VBUS), USBC1.A9 (VBUS), USBC1.B4 (VBUS), USBC1.B9 (VBUS)
- net VD: now also C12.1, C13.1, C14.1, U5.18 (EN), U5.20 (PVIN), U5.21 (PVIN), U5.22 (PVIN)
- net at C26.2: now also R1.2, R20.1, U5.12 (FB); no longer C12.2
- net at C18.1: now also U5.11 (SS/TRK)
- new net: C29.1, U5.6 (BOOT)
- new net: C29.2, L3.2, U5.1 (SW), U5.2 (SW), U5.3 (SW), U5.4 (SW), U5.5 (SW)
- new net: R3.1, R4.2
- new net: R3.2, U5.10 (RT)
- new net: C33.2, U5.8 (VCC)
- new net: R2.2, U5.16 (PGOOD)
Other:
- moved on the sheet: C24

Commit message: feat: updated everything
Parts:
- removed C14: 100uF, Capacitor_SMD:C_Elec_8x10.2, symbol Device:C
- added C14: 100uF, Capacitor_SMD:C_Elec_8x10.2, symbol Device:C_Polarized
Connections:
- net GND: now also C14.2
- net VD: now also C14.1
Changed lines of the file:
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@@
 	)
 	(junction
-		(at 240.03 71.12)
-		(diameter 0)
-		(color 0 0 0 0)
-	)
-	(junction
 		(at 21.59 130.81)
 		(diameter 0)
@@
 	(wire
 		(pts
-			(xy 240.03 71.12) (xy 241.3 71.12)
-		)
-		(stroke
-			(width 0)
-			(type default)
-		)
-	)
-	(wire
-		(pts
 			(xy 189.23 41.91) (xy 223.52 41.91)
 		)
@@
 	(wire
 		(pts
-			(xy 232.41 78.74) (xy 240.03 78.74)
+			(xy 232.41 78.74) (xy 241.3 78.74)
 		)
 		(stroke
@@
 	(wire
 		(pts
-			(xy 232.41 71.12) (xy 240.03 71.12)
+			(xy 232.41 71.12) (xy 241.3 71.12)
 		)
 		(stroke
@@
 	)
 	(symbol
-		(lib_id "Device:C")
-		(at 240.03 74.93 0)
+		(lib_id "power:VDDA")
+		(at 63.5 71.12 180)
 		(unit 1)
 		(exclude_from_sim no)
@@
 		(dnp no)
 		(fields_autoplaced yes)
-		(property "Reference" "C14"
-			(at 243.84 73.6599 0)
+		(property "Reference" "#PWR072"
+			(at 63.5 67.31 0)
 			(effects
 				(font
 					(size 1.27 1.27)
 				)
-				(justify left)
+				(hide yes)
 			)
 		)
-		(property "Value" "100uF"
-			(at 243.84 76.1999 0)
+		(property "Value" "VDDA"
+			(at 63.5 76.2 0)
 			(effects
 				(font
 					(size 1.27 1.27)
 				)
-				(justify left)
 			)
 		)
-		(property "Footprint" "Capacitor_SMD:C_Elec_8x10.2"
-			(at 240.9952 78.74 0)
+		(property "Footprint" ""
+			(at 63.5 71.12 0)
 			(effects
 				(font
@@
 			)
 		)
-		(property "Datasheet" "~"
-			(at 240.03 74.93 0)
+		(property "Datasheet" ""
+			(at 63.5 71.12 0)
 			(effects
 				(font
@@
 			)
 		)
-		(property "Description" "Unpolarized capacitor"
-			(at 240.03 74.93 0)
+		(property "Description" "Power symbol creates a global label with name \"VDDA\""
+			(at 63.5 71.12 0)
 			(effects
 				(font
@@
 		(pin "1"
 		)
-		(pin "2"
-		)
 		(instances
 			(project ""
 				(path "/fe2ec5dd-9620-4cfa-943b-12f58136eb65/b783cc03-ef76-435f-a4cb-a2e41052656e"
-					(reference "C14")
+					(reference "#PWR072")
 					(unit 1)
 				)
@@
 	)
 	(symbol
-		(lib_id "power:VDDA")
-		(at 63.5 71.12 180)
+		(lib_id "power:GND")
+		(at 264.16 35.56 90)
 		(unit 1)
 		(exclude_from_sim no)
@@
 		(dnp no)
 		(fields_autoplaced yes)
-		(property "Reference" "#PWR072"
-			(at 63.5 67.31 0)
+		(property "Reference" "#PWR05"
+			(at 270.51 35.56 0)
 			(effects
 				(font
@@
 			)
 		)
-		(property "Value" "VDDA"
-			(at 63.5 76.2 0)
+		(property "Value" "GND"
+			(at 267.97 35.5599 90)
 			(effects
 				(font
 					(size 1.27 1.27)
 				)
+				(justify right)
 			)
 		)
 		(property "Footprint" ""
-			(at 63.5 71.12 0)
+			(at 264.16 35.56 0)
 			(effects
 				(font
@@
 		)
 		(property "Datasheet" ""
-			(at 63.5 71.12 0)
+			(at 264.16 35.56 0)
 			(effects
 				(font
@@
 			)
 		)
-		(property "Description" "Power symbol creates a global label with name \"VDDA\""
-			(at 63.5 71.12 0)
+		(property "Description" "Power symbol creates a global label with name \"GND\" , ground"
+			(at 264.16 35.56 0)
 			(effects
 				(font
@@
 		)
 		(instances
-			(project ""
+			(project "painter-hat"
 				(path "/fe2ec5dd-9620-4cfa-943b-12f58136eb65/b783cc03-ef76-435f-a4cb-a2e41052656e"
-					(reference "#PWR072")
+					(reference "#PWR05")
 					(unit 1)
 				)
@@
 	(symbol
 		(lib_id "power:GND")
-		(at 264.16 35.56 90)
+		(at 128.27 121.92 0)
 		(unit 1)
 		(exclude_from_sim no)
@@
 		(dnp no)
 		(fields_autoplaced yes)
-		(property "Reference" "#PWR05"
-			(at 270.51 35.56 0)
+		(property "Reference" "#PWR037"
+			(at 128.27 128.27 0)
 			(effects
 				(font
@@
 		)
 		(property "Value" "GND"
-			(at 267.97 35.5599 90)
+			(at 128.27 127 0)
 			(effects
 				(font
 					(size 1.27 1.27)
 				)
-				(justify right)
 			)
 		)
 		(property "Footprint" ""
-			(at 264.16 35.56 0)
+			(at 128.27 121.92 0)
 			(effects
 				(font
@@
 		)
 		(property "Datasheet" ""
-			(at 264.16 35.56 0)
+			(at 128.27 121.92 0)
 			(effects
 				(font
@@
 		)
 		(property "Description" "Power symbol creates a global label with name \"GND\" , ground"
-			(at 264.16 35.56 0)
+			(at 128.27 121.92 0)
 			(effects
 				(font
@@
 		)
 		(instances
-			(project "painter-hat"
+			(project ""
 				(path "/fe2ec5dd-9620-4cfa-943b-12f58136eb65/b783cc03-ef76-435f-a4cb-a2e41052656e"
-					(reference "#PWR05")
+					(reference "#PWR037")
 					(unit 1)
 				)
@@
 	)
 	(symbol
-		(lib_id "power:GND")
-		(at 128.27 121.92 0)
+		(lib_id "Device:C_Polarized")
+		(at 241.3 74.93 0)
 		(unit 1)
 		(exclude_from_sim no)
@@
 		(on_board yes)
 		(dnp no)
-		(fields_autoplaced yes)
-		(property "Reference" "#PWR037"
-			(at 128.27 128.27 0)
+		(property "Reference" "C14"
+			(at 245.11 72.7709 0)
 			(effects
 				(font
 					(size 1.27 1.27)
 				)
-				(hide yes)
+				(justify left)
 			)
 		)
-		(property "Value" "GND"
-			(at 128.27 127 0)
+		(property "Value" "100uF"
+			(at 245.11 75.3109 0)
 			(effects
 				(font
 					(size 1.27 1.27)
 				)
+				(justify left)
 			)
 		)
-		(property "Footprint" ""
-			(at 128.27 121.92 0)
+		(property "Footprint" "Capacitor_SMD:C_Elec_8x10.2"
+			(at 242.2652 78.74 0)
 			(effects
 				(font
@@
 			)
 		)
-		(property "Datasheet" ""
-			(at 128.27 121.92 0)
+		(property "Datasheet" "~"
+			(at 241.3 74.93 0)
 			(effects
 				(font
@@
 			)
 		)
-		(property "Description" "Power symbol creates a global label with name \"GND\" , ground"
-			(at 128.27 121.92 0)
+		(property "Description" "Polarized capacitor"
+			(at 241.3 74.93 0)
 			(effects
 				(font
@@
 		(pin "1"
 		)
+		(pin "2"
+		)
 		(instances
-			(project ""
+			(project "painter-hat"
 				(path "/fe2ec5dd-9620-4cfa-943b-12f58136eb65/b783cc03-ef76-435f-a4cb-a2e41052656e"
-					(reference "#PWR037")
+					(reference "C14")
 					(unit 1)
 				)
